File: Kicad_files/MOTOR.kicad_sch (KiCad schematic)
At the start: 6 parts, among them J1 Screw_Terminal_01x02, J2 Conn_01x08_Pin, J3 Conn_01x15_Pin, J4 Conn_01x15_Pin, U1 NodeMCU1.0(ESP-12E)

Commit message: feat(generated_fab_files): generated_fab_files
Parts:
- added H1, H2, H3, H4: MountingHole, MountingHole:MountingHole_3.2mm_M3, symbol Mechanical:MountingHole
- J3, J4: footprint (none) -> Connector_PinHeader_2.54mm:PinHeader_1x15_P2.54mm_Vertical
Connections:
- net VIN is gone; now on net VCC: J4.1 (Pin_1), U1.15 (VIN)
Other:
- moved on the sheet: J1, J2, J3, J4, PS1, U1
